Commit message: sorry for messy commit, rushed for course project deadline

File: src/onebot_description/urdf/lidar.urdf.xacro (robot description, xacro)
@@ -29,5 +29,5 @@
         <pose>0 0 0 0 0 0</pose>
         <visualize>true</visualize>
-        <update_rate>25</update_rate>
+        <update_rate>15</update_rate>
         <ray>
             <scan>

File: src/onebot_description/urdf/onebot.urdf.xacro (robot description, xacro)
@@ -18,7 +18,8 @@
         <visual>
             <xacro:if value="$(arg mesh_enabled)">
-                <origin xyz="0 0 0" rpy="0 0 0" />
+                <origin xyz="0 0 0" rpy="0 0 3.1415926" />
                 <geometry>
-                    <mesh filename="package://onebot_description/meshes/base_link.dae" />
+                    <!-- <mesh filename="package://onebot_description/meshes/base_link.dae" /> -->
+                    <mesh filename="package://onebot_description/meshes/mice_body_der.stl" />
                 </geometry>
             </xacro:if>
